File: i.mx233stamp/i.MX233.sch (KiCad schematic (older format))
At the start: 28 parts, among them IC1 FSUSB20, J1 MICROSD12P, J2 USBA_RECEPTACLE, J3 USBA-PLUG, P1 CONN_20X2, P2 CONN_20X2, U1 IMX23

Commit message: Added some connections to the pin header and the filters of the sources
Parts:
- removed C1, C11, C7: 10nF, 0402, symbol CAP
- removed C10, C14, C6: 33uF, 0805, symbol CAP
- removed C12, C15, C16, C17, C18, C19, C2, C3, C4, C8: 100nF, 0402, symbol CAP
- removed C13, C5, C9: 1uF, 0603, symbol CAP
- added C? (x2): 20 pF, symbol CAP
- added C?: 50pF, symbol C
- added C?: 1uF, symbol C
- added C? (x2): 8pF, symbol CAP
- added C? (x4): 0.1uF, symbol C
- added L? (x2): 15uH, symbol INDUCTOR
- added P?: CONN_10X2, symbol CONN_10X2
- added P?: CONN_5X2, symbol CONN_5X2
- added Q?: MMDT3904, symbol MMDT3904
- added R?: 10K, symbol R
- added R? (x3): 1K, symbol R
- added R?: 100K, symbol R
- added R? (x3): R, symbol R
- added R? (x5): 47K, symbol R
- added R? (x5): 1.2K, symbol R
- added SW? (x3): SW_PUSH, symbol SW_PUSH
- added X?: 24 MHz, symbol CRYSTAL
- added X?: 32.768 KHz, symbol CRYSTAL
Connections:
- net labels added: GPMI_D15, HPL, HPR, HP_VGND, I2C_SCL, I2C_SDA, LCD_D00, LCD_D01, LCD_D02, LCD_D03, LINE1_INL, LINE1_INR, LRADC0, LRADC1, LRADC2, LRADC3, LRADC4, LRADC5, MIC, PSWITCH, PWM0, PWM1, PWM2, PWM3, PWM4, RTC_XTAL0, RTC_XTAL1, SERIAL_JTAG, SPEAKERN, SPEAKERP, SSP2_CMD, SSP2_DETECT, SSP2_SCK, SSPI_DATA4, SSPI_DETECT, UART1_RX, UART1_TX, VAG, VBUS, VBUS_HOST, VCC, VDD4P2, VDD5V, VDDA, VDDD, VDDIO_3V3, VDDM_2V5, VDD_BATT, VDD_XTAL, V_OUT, XTAL0, XTALI
- wire segments 233 -> 385
- no-connect marks 0 -> 12
Other:
- moved on the sheet: IC1, J1, J2, J3, P1, P2

Commit message: Corrected some signals of uSD card
Parts:
- removed C? (x2): 0.1uF, symbol C
- removed P1: CONN_20X2, header20x2_smd_100mil, symbol CONN_20X2
- removed P?: CONN_10X2, symbol CONN_10X2
- removed P?: CONN_5X2, symbol CONN_5X2
- added BT1: BATTERY, symbol BATTERY
- added C22, C30, C36, C45: 0.01uF, symbol C
- added C23, C24, C28, C31, C32, C37, C41, C44, C46, C47, C49, C51, C55, C56: 0.1uF, symbol C
- added C25, C29, C33, C38, C42, C43, C50: 1uF, symbol C
- added C27, C35, C39: 33uF, symbol C
- added C34: 4.7uF, symbol C
- added C40, C48: 33uF Ceramic, symbol CP1
- added D1: 10BQ015, symbol DIODESCH
- added P3: CONN_25X2, symbol CONN_25X2
- added R1: 1, symbol R
- added R2, R3: 0.1, symbol R
- added R26: 10K, symbol R
- added R27: 22, symbol R
- added RP1, RP2, RP3, RP4, RP5: 22, symbol R_PACK4
- gave numbers to parts that had none: 34
Connections:
- net labels added: LCD_ENABLE1
- net labels removed: MIC, PWM4, SSP2_CMD, SSP2_DETECT, SSP2_SCK, VCC
- wire segments 385 -> 456
- no-connect marks 12 -> 18
Other:
- note added: "BOOT MODES"
- note added: "CRYSTAL'S CIRCUIT"
- note added: "IMX233 PROCESSOR"
- note added: "POWER ON"
- note added: "POWER SUPPLY AND DECOUPLING"
- note added: "RESET CIRCUIT"
- note added: "SERIAL JTAG PINS"
- note added: "SPI SD"
- note added: "USB FIRMWARE RECOVERY"
- note added: "USB HOST AND DEVICE"
- moved on the sheet: C26, C57, C60, IC1, J1, J2, J3, L2, P2, Q1, R10, R11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
