File: TQFP1/i.MX233.sch (KiCad schematic (older format))
At the start: 88 parts, among them IC1 iMX233, J1 MICROSD12P, P3 CONN_5X2, P4 CONN_25X2, P5 CONN_4, Q1 MMDT3904, Q2 SI2305, SW1 SW_PUSH, SW2 SW_PUSH, SW3 SW_PUSH, U4 MC34063, X1 24 MHz

Commit message: PCB placement started
Parts:
- removed C72: 1.5nF, symbol C
- removed C73: 330uF, symbol CAPAPOL
- removed C74, C75: 100uF, symbol CAPAPOL
- removed D2: DIODESCH, symbol DIODESCH
- removed D3: DIODESCH 1AMP, symbol DIODESCH
- removed L2: 170uH, symbol INDUCTOR
- removed L3: 1uH, symbol INDUCTOR
- removed Q2: SI2305, symbol MOS_P
- removed R28: 0.22, symbol R
- removed R29: 10k, symbol R
- removed R30: 180, symbol R
- removed R31: 30k, symbol R
- removed R32: 100K, symbol R
- removed U4: MC34063, symbol MC34063
- added P6: CONN_2X2, symbol CONN_2X2
Connections:
- net labels removed: BATT5V
- wire segments 373 -> 343
Other:
- note added: "Power Supply"
- note removed: "5V BUS"
- note removed: "USB/BATT SWITCH"
- moved on the sheet: J1

Commit message: PCB ADVANCE
Parts:
- removed P4: CONN_25X2, symbol CONN_25X2
- added P1: CONN_8X2, symbol CONN_8X2
- added P2: CONN_12X2, symbol CONN_12X2
Connections:
- wire segments 343 -> 333
