File: TQFP1/i.MX233.sch (KiCad schematic (older format))
At the start: 75 parts, among them IC1 iMX233, J1 MICROSD, P1 CONN_8X2, P2 CONN_12X2, P3 CONN_5X2, P5 CONN_4, P6 CONN_2X2, Q1 MMDT3904, SW1 SW_PUSH, SW2 SW_PUSH, SW3 SW_PUSH, X1 24 MHz

Commit message: PCB Improved
Parts:
- removed C33: 1uF, symbol C
- removed C54: 50pF, symbol C
- removed C55: 0.1uF, symbol C
Connections:
- net labels removed: V_OUT
- wire segments 338 -> 334
- no-connect marks 16 -> 17
Changed lines of the file:
@@
-EESchema Schematic File Version 2  date Tue 15 Feb 2011 11:52:39 AM COT
+EESchema Schematic File Version 2  date Wed 16 Feb 2011 10:56:53 AM COT
 LIBS:microsd
 LIBS:transistor-npn
@@
 Sheet 3 3
 Title ""
-Date "14 feb 2011"
+Date "16 feb 2011"
 Rev ""
 Comp ""
@@
 Comment4 ""
 $EndDescr
+Wire Wire Line
+	2750 12550 3800 12550
+Wire Wire Line
+	7400 11750 7900 11750
 Connection ~ 12900 10700
 Wire Wire Line
@@
 Wire Wire Line
 	6550 10600 6550 10450
-Wire Wire Line
-	7400 11750 8350 11750
-Wire Wire Line
-	8350 11750 8350 11400
 Connection ~ 7900 11750
-Wire Wire Line
-	8350 11000 8350 10600
-Wire Wire Line
-	8350 10600 7100 10600
 Connection ~ 7900 10600
 Wire Wire Line
@@
 Wire Wire Line
 	3300 12550 3300 12650
-Connection ~ 3450 12150
-Wire Wire Line
-	3800 12150 2750 12150
-Connection ~ 3450 12550
-Wire Wire Line
-	2750 12550 3800 12550
 Connection ~ 3100 12550
 Connection ~ 3100 12150
@@
 Wire Wire Line
 	1450 1750 1550 1750
-Wire Wire Line
-	8050 7600 6400 7600
-Connection ~ 7800 7600
-Wire Wire Line
-	7800 8000 7800 8150
 Wire Wire Line
 	1900 10700 1900 10950
@@
 	13850 10700 13850 10650
 Connection ~ 13850 10650
+Wire Wire Line
+	7900 10600 7100 10600
+Wire Wire Line
+	3800 12150 2750 12150
+NoConn ~ 6400 7600
 $Comp
 L GND #PWR012
@@
 $EndComp
 $Comp
-L C C55
-U 1 1 4D42D636
-P 8350 11200
-F 0 "C55" H 8400 11300 50  0000 L CNN
-F 1 "0.1uF" H 8400 11100 50  0000 L CNN
-	1    8350 11200
-	1    0    0    -1
-$EndComp
-$Comp
 L GND #PWR053
 U 1 1 4D42D635
@@
 F 1 "33uF" H 3850 12250 50  0000 L CNN
 	1    3800 12350
-	1    0    0    -1
-$EndComp
-$Comp
-L C C33
-U 1 1 4D42D62B
-P 3450 12350
-F 0 "C33" H 3500 12450 50  0000 L CNN
-F 1 "1uF" H 3500 12250 50  0000 L CNN
-	1    3450 12350
 	1    0    0    -1
 $EndComp
@@
 Text Label 6638 7750 0    60   ~ 0
 VAG
-Text Label 8050 7600 0    60   ~ 0
-V_OUT
-$Comp
-L GND #PWR078
-U 1 1 4D4053BE
-P 7800 8150
-F 0 "#PWR078" H 7800 8150 30  0001 C CNN
-F 1 "GND" H 7800 8080 30  0001 C CNN
-	1    7800 8150
-	1    0    0    -1
-$EndComp
-$Comp
-L C C54
-U 1 1 4D4053B0
-P 7800 7800
-F 0 "C54" H 7850 7900 50  0000 L CNN
-F 1 "50pF" H 7850 7700 50  0000 L CNN
-	1    7800 7800
-	1    0    0    -1
-$EndComp
 $Comp
 L GND #PWR079

Commit message: Corrected PCB errors in the memory, added a MAX-232 to the UART Voltage levels and added 4 leds...
Parts:
- added C1, C2, C3, C5: 0.1uF, symbol C
- added C4: .1uF, symbol C
- added D2, D3, D4, D5: LED, symbol LED
- added P4: CONN_4, symbol CONN_4
- added R28, R30, R31, R9: 1k, symbol R
- added R29: 47k, symbol R
- added U1: ADM3101E, symbol ADM3101E
Connections:
- net labels added: LCD_D04, LCD_D05, LCD_D06, LCD_D07, RX, TX
- net labels removed: GNDPWR
- wire segments 334 -> 370
- no-connect marks 17 -> 18
Other:
- moved on the sheet: RP3, RP4

Commit message: Fixed ADM Signals and organize schematic
Connections:
- wire segments 370 -> 368
Other:
- note added: "ADM3101E CIRCUIT"
- note added: "UART CONNECTOR"
- moved on the sheet: BT1, C1, C2, C22, C23, C24, C25, C26, C27, C28, C29, C3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
