File: TQFP1/i.MX233.sch (KiCad schematic (older format))
At the start: 88 parts, among them IC1 iMX233, J1 MICROSD, P1 CONN_8X2, P2 CONN_12X2, P3 CONN_5X2, P4 CONN_4, P5 CONN_4, P6 CONN_2X2, Q1 MMDT3904, SW1 SW_PUSH, SW2 SW_PUSH, SW3 SW_PUSH, U1 ADM3101E, X1 24 MHz

Commit message: PCB labels, improvements 15/04/11
Parts:
- removed P4, P5: CONN_4, symbol CONN_4
- removed P6: CONN_2X2, symbol CONN_2X2
- added J2: JACK-PLUG0, con-jack-SPC4077, symbol JACK-PLUG0
- added JP3: JUMPER, symbol JUMPER
- added L2: HZ0805D152R-10 (1500 ohm), symbol INDUCTOR
- added P6: CONN_2, symbol CONN_2
- added P?: CONN_4X2, symbol CONN_4X2
- added R32: 47k, symbol R
- R13, R16: value 1K -> 47k
- R17, R18, R19, R20, R21: value 1.2K -> 10K
Connections:
- net labels added: D03

Commit message: Some PCB and boot changes
Parts:
- removed P3: CONN_5X2, symbol CONN_5X2
- removed R20, R21: 10K, symbol R
- added JP1, JP2: JUMPER, symbol JUMPER
- added R33: 0, symbol R
- R11, R12, R14: value 47K -> 1.5k
- R15: value 47K -> 11k
- R17, R18, R19: value 10K -> 11k
- gave numbers to parts that had none: 1
Connections:
- wire segments 368 -> 363
Other:
- moved on the sheet: D4, J2, P6, R10, R30, R32

Commit message: More changes to the PCB
Parts:
- R13, R16: value 47k -> 1k
Changed lines of the file:
@@
-EESchema Schematic File Version 2  date Thu 21 Apr 2011 06:26:39 PM COT
+EESchema Schematic File Version 2  date Mon 25 Apr 2011 11:56:53 AM COT
+LIBS:con-jack
+LIBS:adm3101e
+LIBS:microsd
+LIBS:transistor-npn
+LIBS:ipc-7351-transistor
+LIBS:switch-misc
 LIBS:power
 LIBS:device
@@
 LIBS:contrib
 LIBS:valves
+LIBS:micron_ddr_512Mb
+LIBS:iMX23
+LIBS:sdmmc
+LIBS:usbconn
+LIBS:fsusb20
+LIBS:r_pack2
+LIBS:pasives-connectors
+LIBS:EEPROM
+LIBS:PWR
+LIBS:m25p32
+LIBS:PROpendous-cache
+LIBS:w_analog
 LIBS:i.mx233stamp-cache
 EELAYER 25  0
@@
 Sheet 3 3
 Title ""
-Date "21 apr 2011"
+Date "25 apr 2011"
 Rev ""
 Comp ""
@@
 P 9950 2800
 F 0 "R13" V 10030 2800 50  0000 C CNN
-F 1 "47k" V 9950 2800 50  0000 C CNN
+F 1 "1k" V 9950 2800 50  0000 C CNN
 	1    9950 2800
 	0    1    1    0
@@
 P 10450 3100
 F 0 "R16" V 10530 3100 50  0000 C CNN
-F 1 "47k" V 10450 3100 50  0000 C CNN
+F 1 "1k" V 10450 3100 50  0000 C CNN
 	1    10450 3100
 	1    0    0    -1
