File: PCB/TQFP1/USB.sch (KiCad schematic (older format))
At the start: 1 part, among them U4 GL850G

Commit message: primera conexion bus usb
Connections:
- net USB_DM0: now reaches U4.25 (DM0)
- net USB_DP0: now reaches U4.26 (DP0)
Changed lines of the file:
@@
-EESchema Schematic File Version 2  date Fri 05 Aug 2011 08:43:14 AM COT
+EESchema Schematic File Version 2  date Fri 05 Aug 2011 09:02:43 AM COT
+LIBS:con-jack
+LIBS:adm3101e
+LIBS:microsd
 LIBS:transistor-npn
 LIBS:ipc-7351-transistor
@@
 Comment4 ""
 $EndDescr
+Wire Wire Line
+	6900 2950 6600 2950
+Wire Wire Line
+	6900 2850 6600 2850
+Text HLabel 6900 2950 2    60   3State ~ 0
+USB_DM0
+Text HLabel 6900 2850 2    60   3State ~ 0
+USB_DP0
 $Comp
 L GL850G U4

Commit message: hub
Parts:
- added C10, C11, C13, C15, C16, C9: 100nF, SM0603, symbol C
- added C12, C8: 10nF, SM0603, symbol C
- added C14: 4.7uF, SM1206, symbol C
- added C6, C7: 8pF, SM0603, symbol C
- added L3, L4, L5, L6: SRF2012, SRF2012, symbol SRF2012
- added L7: 2A 120 ohm, symbol INDUCTOR
- added R20: 1M, SM0603, symbol R
- added R21: 100k, SM0603, symbol R
- added R36: 680 1%, SM0603, symbol R
- added X2: 12MHz, symbol CRYSTAL
Connections:
- net labels added: GND, USBH_P33V, USBH_P33VD, USB_DM1, USB_DM2, USB_DM3, USB_DM4, USB_DP1, USB_DP2, USB_DP3, USB_DP4, VDD5V, X1, X2
- wire segments 2 -> 90
Other:
- note added: "andres.calderon@emqbit.com\n"
- moved on the sheet: U4
