File: PCB/i.mx233stamp-bga/DDR1.sch (KiCad schematic (older format))
At the start: 17 parts, among them U2 MT46V32M16TG, U3 M25P32

Commit message: clean-up
Connections:
- net labels added: SSPI_DATA4
- net labels removed: SSPI_DATA3
Changed lines of the file:
@@
-EESchema Schematic File Version 2  date vie 28 ene 2011 11:40:08 COT
+EESchema Schematic File Version 2  date mié 02 feb 2011 14:04:32 COT
 LIBS:transistor-npn
 LIBS:ipc-7351-transistor
@@
 LIBS:PWR
 LIBS:m25p32
+LIBS:w_analog
 LIBS:i.mx233stamp-cache
 EELAYER 24  0
@@
 Sheet 2 3
 Title ""
-Date "28 jan 2011"
+Date "2 feb 2011"
 Rev ""
 Comp ""
@@
 $EndComp
 $Comp
-L GND #PWR82
+L GND #PWR01
 U 1 1 4D418353
 P 6500 4350
-F 0 "#PWR82" H 6500 4350 30  0001 C CNN
+F 0 "#PWR01" H 6500 4350 30  0001 C CNN
 F 1 "GND" H 6500 4280 30  0001 C CNN
 	1    6500 4350
@@
 DDR_CKE
 $Comp
-L GND #PWR92
+L GND #PWR02
 U 1 1 4D417AF1
 P 10800 2750
-F 0 "#PWR92" H 10800 2750 30  0001 C CNN
+F 0 "#PWR02" H 10800 2750 30  0001 C CNN
 F 1 "GND" H 10800 2680 30  0001 C CNN
 	1    10800 2750
@@
 $EndComp
 $Comp
-L VDDM_2V5 #PWR91
+L VDDM_2V5 #PWR03
 U 1 1 4D417ACD
 P 10800 1450
-F 0 "#PWR91" H 10800 1550 30  0001 C CNN
+F 0 "#PWR03" H 10800 1550 30  0001 C CNN
 F 1 "VDDM_2V5" H 10800 1550 30  0000 C CNN
 	1    10800 1450
@@
 $EndComp
 $Comp
-L VDDM_2V5 #PWR83
+L VDDM_2V5 #PWR04
 U 1 1 4D4179A4
 P 7250 800
-F 0 "#PWR83" H 7250 900 30  0001 C CNN
+F 0 "#PWR04" H 7250 900 30  0001 C CNN
 F 1 "VDDM_2V5" H 7250 900 30  0000 C CNN
 	1    7250 800
@@
 $EndComp
 $Comp
-L VDDM_2V5 #PWR89
+L VDDM_2V5 #PWR05
 U 1 1 4D417999
 P 10200 800
-F 0 "#PWR89" H 10200 900 30  0001 C CNN
+F 0 "#PWR05" H 10200 900 30  0001 C CNN
 F 1 "VDDM_2V5" H 10200 900 30  0000 C CNN
 	1    10200 800
@@
 $EndComp
 $Comp
-L GND #PWR84
+L GND #PWR06
 U 1 1 4D41792B
 P 7550 1500
-F 0 "#PWR84" H 7550 1500 30  0001 C CNN
+F 0 "#PWR06" H 7550 1500 30  0001 C CNN
 F 1 "GND" H 7550 1430 30  0001 C CNN
 	1    7550 1500
@@
 $EndComp
 $Comp
-L GND #PWR88
+L GND #PWR07
 U 1 1 4D417882
 P 9600 1500
-F 0 "#PWR88" H 9600 1500 30  0001 C CNN
+F 0 "#PWR07" H 9600 1500 30  0001 C CNN
 F 1 "GND" H 9600 1430 30  0001 C CNN
 	1    9600 1500
@@
 SSPI_DATA0
 Text HLabel 7700 6150 0    60   Input ~ 0
-SSPI_DATA3
-$Comp
-L GND #PWR90
+SSPI_DATA4
+$Comp
+L GND #PWR08
 U 1 1 4D409664
 P 10400 6050
-F 0 "#PWR90" H 10400 6050 30  0001 C CNN
+F 0 "#PWR08" H 10400 6050 30  0001 C CNN
 F 1 "GND" H 10400 5980 30  0001 C CNN
 	1    10400 6050
@@
 $EndComp
 $Comp
-L VDDIO_3V3 #PWR87
+L VDDIO_3V3 #PWR09
 U 1 1 4D409635
 P 9500 5950
-F 0 "#PWR87" H 9500 6050 30  0001 C CNN
+F 0 "#PWR09" H 9500 6050 30  0001 C CNN
 F 1 "VDDIO_3V3" H 9500 6050 30  0000 C CNN
 	1    9500 5950
@@
 $EndComp
 $Comp
-L GND #PWR85
+L GND #PWR010
 U 1 1 4D409619
 P 7650 6700
-F 0 "#PWR85" H 7650 6700 30  0001 C CNN
+F 0 "#PWR010" H 7650 6700 30  0001 C CNN
 F 1 "GND" H 7650 6630 30  0001 C CNN
 	1    7650 6700
@@
 DDR_WEN
 $Comp
-L GND #PWR86
+L GND #PWR011
 U 1 1 4D319D50
 P 8300 5050
-F 0 "#PWR86" H 8300 5050 30  0001 C CNN
+F 0 "#PWR011" H 8300 5050 30  0001 C CNN
 F 1 "GND" H 8300 4980 30  0001 C CNN
 	1    8300 5050
