File: PCB/i.mx233stamp-bga/i.MX233.sch (KiCad schematic (older format))
At the start: 80 parts, among them IC1 FSUSB20, J1 MICROSD12P, J2 USBA_RECEPTACLE, J3 USBA-PLUG, P1 CONN_20X2, P2 CONN_20X2, P3 CONN_5X2, Q1 MMDT3904, SW1 SW_PUSH, SW2 SW_PUSH, SW3 SW_PUSH, U1 IMX23, X1 24 MHz, X2 32.768 KHz

Commit message: clean-up
Parts:
- removed P1: CONN_20X2, header20x2_smd_100mil, symbol CONN_20X2
- removed P3: CONN_5X2, symbol CONN_5X2
- added C72: 1.5nF, symbol C
- added C73: 330uF, symbol CAPAPOL
- added C74: 100uF, symbol CAPAPOL
- added D2: DIODESCH, symbol DIODESCH
- added D3: DIODESCH 1 AMP, symbol DIODESCH
- added L3: 170uH, symbol INDUCTOR
- added L4: 1u, symbol INDUCTOR
- added P3: CONN_25X2, symbol CONN_25X2
- added Q2: SI2305, symbol MOSFET_P
- added R26, R30: 10K, symbol R
- added R27: 22, symbol R
- added R28: 0.22, symbol R
- added R29: 180, symbol R
- added R31: 30K, symbol R
- added R32: 100K, symbol R
- added RP1, RP2, RP3, RP4, RP5: 22, symbol R_PACK4
- added U4: MC34063, symbol MC34063
Connections:
- net labels added: BATT5V, LCD_ENABLE1
- wire segments 425 -> 494
Other:
- note added: "5V BUS"
- note added: "BUS/BATT SWITCH"
- moved on the sheet: J1, P2, R10, R11, R12, R14, R15, R17, R18, R19, R20, R21
