File: PCB/i.mx233stamp-bga/i.mx233stamp.sch (KiCad schematic (older format))
At the start: 0 parts

Commit message: clean-up
Changed lines of the file:
@@
-EESchema Schematic File Version 2  date mié 02 feb 2011 11:17:26 COT
+EESchema Schematic File Version 2  date mié 02 feb 2011 14:04:32 COT
 LIBS:transistor-npn
 LIBS:ipc-7351-transistor
@@
 LIBS:PWR
 LIBS:m25p32
+LIBS:w_analog
 LIBS:i.mx233stamp-cache
 EELAYER 24  0
@@
 Sheet 1 3
 Title ""
-Date "28 jan 2011"
+Date "2 feb 2011"
 Rev ""
 Comp ""
@@
 F15 "DDR_RASN" I L 5250 2950 60
 F16 "DDR_WEN" I L 5250 2750 60
-F17 "SSPI_DATA3" I L 5250 2050 60
+F17 "SSPI_DATA4" I L 5250 2050 60
 F18 "SSPI_DATA2" I L 5250 1950 60
 F19 "SSPI_SCK" I L 5250 2150 60
@@
 F15 "DDR_BA1" O R 4750 4050 60
 F16 "DDR_BA0" O R 4750 3950 60
-F17 "SSPI_DATA3" O R 4750 2050 60
+F17 "SSPI_DATA4" O R 4750 2050 60
 F18 "SSPI_SCK" O R 4750 2150 60
 F19 "SSPI_CMD" O R 4750 2250 60
