File: PCB/i.mx233stamp/DDR1.sch (KiCad schematic (older format))
At the start: 17 parts, among them U2 MT46V32M16TG, U3 M25P32

Commit message: clean-up
Parts:
- added R34, R35: 0, symbol R
- added R7: 47k, symbol R
- added R8: 10k, symbol R
- R22: value R -> 110
Connections:
- net labels added: GPMI_D00, GPMI_D01, GPMI_D02, GPMI_D03, GPMI_D04, GPMI_RDY1, GPMI_WRN
- net labels removed: SSPI_CMD, SSPI_DATA0, SSPI_DATA1, SSPI_DATA2, SSPI_DATA4, SSPI_SCK
- wire segments 136 -> 142
Other:
- moved on the sheet: R23
Changed lines of the file:
@@
-EESchema Schematic File Version 2  date mié 02 feb 2011 14:04:32 COT
+EESchema Schematic File Version 2  date Fri 05 Aug 2011 02:31:32 PM COT
+LIBS:con-jack
+LIBS:adm3101e
+LIBS:microsd
 LIBS:transistor-npn
 LIBS:ipc-7351-transistor
@@
 LIBS:PWR
 LIBS:m25p32
+LIBS:PROpendous-cache
 LIBS:w_analog
+LIBS:gl850g
+LIBS:srf2012
 LIBS:i.mx233stamp-cache
-EELAYER 24  0
+EELAYER 25  0
 EELAYER END
 $Descr A4 11700 8267
-Sheet 2 3
+encoding utf-8
+Sheet 3 4
 Title ""
-Date "2 feb 2011"
+Date "5 aug 2011"
 Rev ""
 Comp ""
@@
 Comment4 ""
 $EndDescr
-Text Notes 5850 5500 0    60   ~ 0
-SPI FLASH
+Wire Wire Line
+	7050 6000 7100 6000
+Wire Wire Line
+	7600 5750 7650 5750
+Connection ~ 7650 6000
+Wire Wire Line
+	8200 6150 7650 6150
+Wire Wire Line
+	7650 6150 7650 5750
+Connection ~ 7950 6150
+Wire Wire Line
+	7950 6050 7950 6150
+Wire Wire Line
+	5850 4500 5850 4300
+Wire Wire Line
+	6500 3900 7250 3900
 Wire Notes Line
 	5750 5350 5750 7150
@@
 Wire Wire Line
 	6700 3300 7250 3300
-Wire Wire Line
-	7250 3800 6500 3800
 Connection ~ 10800 1500
 Wire Wire Line
@@
 Wire Wire Line
 	7700 6350 8200 6350
-Wire Wire Line
-	7700 6150 8200 6150
 Connection ~ 8550 1500
 Connection ~ 8350 1500
@@
 Connection ~ 10800 2700
 Wire Wire Line
-	6500 4300 6500 4350
-Wire Wire Line
 	6700 3400 7250 3400
 Wire Wire Line
 	6700 3600 7250 3600
-Wire Wire Line
-	6750 3900 7250 3900
 Wire Wire Line
 	9450 3400 10000 3400
@@
 Wire Notes Line
 	11150 7150 5750 7150
+Wire Wire Line
+	5850 3800 7250 3800
+Wire Wire Line
+	7050 5750 7100 5750
+Wire Wire Line
+	7600 6000 7650 6000
+$Comp
+L R R35
+U 1 1 4DACFF24
+P 7350 6000
+F 0 "R35" V 7430 6000 50  0000 C CNN
+F 1 "0" V 7350 6000 50  0000 C CNN
+	1    7350 6000
+	0    1    1    0
+$EndComp
+$Comp
+L R R34
+U 1 1 4DACFF20
+P 7350 5750
+F 0 "R34" V 7430 5750 50  0000 C CNN
+F 1 "0" V 7350 5750 50  0000 C CNN
+	1    7350 5750
+	0    1    1    0
+$EndComp
+Text HLabel 7050 5750 0    60   Input ~ 0
+GPMI_D03
+$Comp
+L VDDIO_3V3 #PWR18
+U 1 1 4D7E71FF
+P 7950 5550
+F 0 "#PWR18" H 7950 5650 30  0001 C CNN
+F 1 "VDDIO_3V3" H 7950 5650 30  0000 C CNN
+	1    7950 5550
+	1    0    0    -1
+$EndComp
+$Comp
+L R R8
+U 1 1 4D7E71FA
+P 7950 5800
+F 0 "R8" V 8030 5800 50  0000 C CNN
+F 1 "10k" V 7950 5800 50  0000 C CNN
+	1    7950 5800
+	1    0    0    -1
+$EndComp
+$Comp
+L VDDM_2V5 #PWR14
+U 1 1 4D7E6BF9
+P 6000 3900
+F 0 "#PWR14" H 6000 4000 30  0001 C CNN
+F 1 "VDDM_2V5" H 5950 3950 30  0000 C CNN
+	1    6000 3900
+	1    0    0    -1
+$EndComp
+$Comp
+L R R7
+U 1 1 4D7E6AED
+P 6250 3900
+F 0 "R7" V 6330 3900 50  0000 C CNN
+F 1 "47k" V 6250 3900 50  0000 C CNN
+	1    6250 3900
+	0    1    1    0
+$EndComp
+Text Notes 5850 5500 0    60   ~ 0
+SPI FLASH
 Text Notes 5850 750  0    60   ~ 0
 DDR RAM
@@
 P 5950 3450
 F 0 "R22" V 6030 3450 50  0000 C CNN
-F 1 "R" V 5950 3450 50  0000 C CNN
+F 1 "110" V 5950 3450 50  0000 C CNN
 	1    5950 3450
 	1    0    0    -1
@@
 Text Label 2200 4850 0    60   ~ 0
 DDR_CKE
-Text Label 2200 4550 0    60   ~ 0
-DDR_CKE
-Text Label 2200 4550 0    60   ~ 0
+Text Label 2250 4550 0    60   ~ 0
 DDR_CASN
 Text Label 2200 4950 0    60   ~ 0
@@
 L R R23
 U 1 1 4D418363
-P 6500 4050
-F 0 "R23" V 6580 4050 50  0000 C CNN
-F 1 "47K" V 6500 4050 50  0000 C CNN
-	1    6500 4050
-	1    0    0    -1
-$EndComp
-$Comp
-L GND #PWR01
+P 5850 4050
+F 0 "R23" V 5930 4050 50  0000 C CNN
+F 1 "47K" V 5850 4050 50  0000 C CNN
+	1    5850 4050
+	1    0    0    -1
+$EndComp
+$Comp
+L GND #PWR13
 U 1 1 4D418353
-P 6500 4350
-F 0 "#PWR01" H 6500 4350 30  0001 C CNN
-F 1 "GND" H 6500 4280 30  0001 C CNN
-	1    6500 4350
+P 5850 4500
+F 0 "#PWR13" H 5850 4500 30  0001 C CNN
+F 1 "GND" H 5850 4430 30  0001 C CNN
+	1    5850 4500
 	1    0    0    -1
 $EndComp
@@
 DDR_CKE
 $Comp
-L GND #PWR02
+L GND #PWR25
 U 1 1 4D417AF1
 P 10800 2750
-F 0 "#PWR02" H 10800 2750 30  0001 C CNN
+F 0 "#PWR25" H 10800 2750 30  0001 C CNN
 F 1 "GND" H 10800 2680 30  0001 C CNN
 	1    10800 2750
@@
 $EndComp
 $Comp
-L VDDM_2V5 #PWR03
+L VDDM_2V5 #PWR24
 U 1 1 4D417ACD
 P 10800 1450
-F 0 "#PWR03" H 10800 1550 30  0001 C CNN
+F 0 "#PWR24" H 10800 1550 30  0001 C CNN
 F 1 "VDDM_2V5" H 10800 1550 30  0000 C CNN
 	1    10800 1450
@@
 $EndComp
 $Comp
-L VDDM_2V5 #PWR04
+L VDDM_2V5 #PWR15
 U 1 1 4D4179A4
 P 7250 800
-F 0 "#PWR04" H 7250 900 30  0001 C CNN
+F 0 "#PWR15" H 7250 900 30  0001 C CNN
 F 1 "VDDM_2V5" H 7250 900 30  0000 C CNN
 	1    7250 800
@@
 $EndComp
 $Comp
-L VDDM_2V5 #PWR05
+L VDDM_2V5 #PWR22
 U 1 1 4D417999
 P 10200 800
-F 0 "#PWR05" H 10200 900 30  0001 C CNN
+F 0 "#PWR22" H 10200 900 30  0001 C CNN
 F 1 "VDDM_2V5" H 10200 900 30  0000 C CNN
 	1    10200 800
@@
 $EndComp
 $Comp
-L GND #PWR06
+L GND #PWR16
 U 1 1 4D41792B
 P 7550 1500
-F 0 "#PWR06" H 7550 1500 30  0001 C CNN
+F 0 "#PWR16" H 7550 1500 30  0001 C CNN
 F 1 "GND" H 7550 1430 30  0001 C CNN
 	1    7550 1500
@@
 $EndComp
 $Comp
-L GND #PWR07
+L GND #PWR21
 U 1 1 4D417882
 P 9600 1500
-F 0 "#PWR07" H 9600 1500 30  0001 C CNN
+F 0 "#PWR21" H 9600 1500 30  0001 C CNN
 F 1 "GND" H 9600 1430 30  0001 C CNN
 	1    9600 1500
@@
 $EndComp
 Text HLabel 9850 6250 2    60   Input ~ 0
-SSPI_DATA2
+GPMI_D02
 Text HLabel 9850 6350 2    60   Input ~ 0
-SSPI_SCK
+GPMI_WRN
 Text HLabel 9850 6450 2    60   Input ~ 0
-SSPI_CMD
+GPMI_RDY1
 Text HLabel 7700 6350 0    60   Input ~ 0
-SSPI_DATA1
+GPMI_D01
 Text HLabel 7700 6250 0    60   Input ~ 0
-SSPI_DATA0
-Text HLabel 7700 6150 0    60   Input ~ 0
-SSPI_DATA4
-$Comp
-L GND #PWR08
+GPMI_D00
+Text HLabel 7050 6000 0    60   Input ~ 0
+GPMI_D04
+$Comp
+L GND #PWR23
 U 1 1 4D409664
 P 10400 6050
-F 0 "#PWR08" H 10400 6050 30  0001 C CNN
+F 0 "#PWR23" H 10400 6050 30  0001 C CNN
 F 1 "GND" H 10400 5980 30  0001 C CNN
 	1    10400 6050
@@
 $EndComp
 $Comp
-L VDDIO_3V3 #PWR09
+L VDDIO_3V3 #PWR20
 U 1 1 4D409635
 P 9500 5950
-F 0 "#PWR09" H 9500 6050 30  0001 C CNN
+F 0 "#PWR20" H 9500 6050 30  0001 C CNN
 F 1 "VDDIO_3V3" H 9500 6050 30  0000 C CNN
 	1    9500 5950
@@
 $EndComp
 $Comp
-L GND #PWR010
+L GND #PWR17
 U 1 1 4D409619
 P 7650 6700
-F 0 "#PWR010" H 7650 6700 30  0001 C CNN
+F 0 "#PWR17" H 7650 6700 30  0001 C CNN
 F 1 "GND" H 7650 6630 30  0001 C CNN
 	1    7650 6700
@@
 DDR_WEN
 $Comp
-L GND #PWR011
+L GND #PWR19
 U 1 1 4D319D50
 P 8300 5050
-F 0 "#PWR011" H 8300 5050 30  0001 C CNN
+F 0 "#PWR19" H 8300 5050 30  0001 C CNN
 F 1 "GND" H 8300 4980 30  0001 C CNN
 	1    8300 5050

Commit message: Cambios en los footprints, adición de conectores USB host, organización de señales en los conectores
Parts:
- U2: footprint TSOP-66 -> TSOP66_JEDEC_DDR_SDRAM
- U3: footprint (none) -> SO16W
Changed lines of the file:
@@
-EESchema Schematic File Version 2  date Mon 08 Aug 2011 07:05:33 AM COT
+EESchema Schematic File Version 2  date Tue 09 Aug 2011 03:40:13 PM COT
 LIBS:con-jack
 LIBS:adm3101e
@@
 LIBS:gl850g
 LIBS:srf2012
+LIBS:rclamp0502b
 LIBS:i.mx233stamp-cache
-EELAYER 25  0
+EELAYER 24  0
 EELAYER END
 $Descr A4 11700 8267
@@
 Sheet 3 4
 Title ""
-Date "8 aug 2011"
+Date "9 aug 2011"
 Rev ""
 Comp ""
@@
 GPMI_D03
 $Comp
-L VDDIO_3V3 #PWR013
+L VDDIO_3V3 #PWR023
 U 1 1 4D7E71FF
 P 7950 5550
-F 0 "#PWR013" H 7950 5650 30  0001 C CNN
+F 0 "#PWR023" H 7950 5650 30  0001 C CNN
 F 1 "VDDIO_3V3" H 7950 5650 30  0000 C CNN
 	1    7950 5550
@@
 $EndComp
 $Comp
-L VDDM_2V5 #PWR014
+L VDDM_2V5 #PWR024
 U 1 1 4D7E6BF9
 P 6000 3900
-F 0 "#PWR014" H 6000 4000 30  0001 C CNN
+F 0 "#PWR024" H 6000 4000 30  0001 C CNN
 F 1 "VDDM_2V5" H 5950 3950 30  0000 C CNN
 	1    6000 3900
@@
 $EndComp
 $Comp
-L GND #PWR015
+L GND #PWR025
 U 1 1 4D418353
 P 5850 4500
-F 0 "#PWR015" H 5850 4500 30  0001 C CNN
+F 0 "#PWR025" H 5850 4500 30  0001 C CNN
 F 1 "GND" H 5850 4430 30  0001 C CNN
 	1    5850 4500
@@
 DDR_CKE
 $Comp
-L GND #PWR016
+L GND #PWR026
 U 1 1 4D417AF1
 P 10800 2750
-F 0 "#PWR016" H 10800 2750 30  0001 C CNN
+F 0 "#PWR026" H 10800 2750 30  0001 C CNN
 F 1 "GND" H 10800 2680 30  0001 C CNN
 	1    10800 2750
@@
 $EndComp
 $Comp
-L VDDM_2V5 #PWR017
+L VDDM_2V5 #PWR027
 U 1 1 4D417ACD
 P 10800 1450
-F 0 "#PWR017" H 10800 1550 30  0001 C CNN
+F 0 "#PWR027" H 10800 1550 30  0001 C CNN
 F 1 "VDDM_2V5" H 10800 1550 30  0000 C CNN
 	1    10800 1450
@@
 $EndComp
 $Comp
-L VDDM_2V5 #PWR018
+L VDDM_2V5 #PWR028
 U 1 1 4D4179A4
 P 7250 800
-F 0 "#PWR018" H 7250 900 30  0001 C CNN
+F 0 "#PWR028" H 7250 900 30  0001 C CNN
 F 1 "VDDM_2V5" H 7250 900 30  0000 C CNN
 	1    7250 800
@@
 $EndComp
 $Comp
-L VDDM_2V5 #PWR019
+L VDDM_2V5 #PWR029
 U 1 1 4D417999
 P 10200 800
-F 0 "#PWR019" H 10200 900 30  0001 C CNN
+F 0 "#PWR029" H 10200 900 30  0001 C CNN
 F 1 "VDDM_2V5" H 10200 900 30  0000 C CNN
 	1    10200 800
@@
 $EndComp
 $Comp
-L GND #PWR020
+L GND #PWR030
 U 1 1 4D41792B
 P 7550 1500
-F 0 "#PWR020" H 7550 1500 30  0001 C CNN
+F 0 "#PWR030" H 7550 1500 30  0001 C CNN
 F 1 "GND" H 7550 1430 30  0001 C CNN
 	1    7550 1500
@@
 $EndComp
 $Comp
-L GND #PWR021
+L GND #PWR031
 U 1 1 4D417882
 P 9600 1500
-F 0 "#PWR021" H 9600 1500 30  0001 C CNN
+F 0 "#PWR031" H 9600 1500 30  0001 C CNN
 F 1 "GND" H 9600 1430 30  0001 C CNN
 	1    9600 1500
@@
 GPMI_D04
 $Comp
-L GND #PWR022
+L GND #PWR032
 U 1 1 4D409664
 P 10400 6050
-F 0 "#PWR022" H 10400 6050 30  0001 C CNN
+F 0 "#PWR032" H 10400 6050 30  0001 C CNN
 F 1 "GND" H 10400 5980 30  0001 C CNN
 	1    10400 6050
@@
 $EndComp
 $Comp
-L VDDIO_3V3 #PWR023
+L VDDIO_3V3 #PWR033
 U 1 1 4D409635
 P 9500 5950
-F 0 "#PWR023" H 9500 6050 30  0001 C CNN
+F 0 "#PWR033" H 9500 6050 30  0001 C CNN
 F 1 "VDDIO_3V3" H 9500 6050 30  0000 C CNN
 	1    9500 5950
@@
 $EndComp
 $Comp
-L GND #PWR024
+L GND #PWR034
 U 1 1 4D409619
 P 7650 6700
-F 0 "#PWR024" H 7650 6700 30  0001 C CNN
+F 0 "#PWR034" H 7650 6700 30  0001 C CNN
 F 1 "GND" H 7650 6630 30  0001 C CNN
 	1    7650 6700
@@
 F 0 "U3" H 8650 6350 60  0000 C CNN
 F 1 "M25P32" H 8600 6450 60  0000 C CNN
+F 2 "SO16W" H 8800 6200 60  0001 C CNN
 	1    8800 6200
 	1    0    0    -1
@@
 DDR_WEN
 $Comp
-L GND #PWR025
+L GND #PWR035
 U 1 1 4D319D50
 P 8300 5050
-F 0 "#PWR025" H 8300 5050 30  0001 C CNN
+F 0 "#PWR035" H 8300 5050 30  0001 C CNN
 F 1 "GND" H 8300 4980 30  0001 C CNN
 	1    8300 5050
@@
 F 0 "U2" H 8350 3300 70  0000 C CNN
 F 1 "MT46V32M16TG" H 8350 3100 70  0000 C CNN
-F 2 "TSOP-66" H 8350 3200 60  0001 C CNN
+F 2 "TSOP66_JEDEC_DDR_SDRAM" H 8350 3200 60  0001 C CNN
 	1    8350 3200
 	1    0    0    -1
