File: PCB/i.mx233stamp/i.MX233.sch (KiCad schematic (older format))
At the start: 100 parts, among them IC1 FSUSB20, J1 MICROSD12P, J2 USBA_RECEPTACLE, J3 USBA-PLUG, P2 CONN_20X2, P3 CONN_25X2, Q1 MMDT3904, Q2 SI2305, SW1 SW_PUSH, SW2 SW_PUSH, SW3 SW_PUSH, U1 IMX23, U4 MC34063, X1 24 MHz, X2 32.768 KHz

Commit message: clean-up
Parts:
- removed C20: 100nF, 0402, symbol CAP
- removed C21: 1uF, 0603, symbol CAP
- removed C33: 1uF, symbol C
- removed C54: 50pF, symbol C
- removed C55: 0.1uF, symbol C
- removed C58, C59: 8pF, symbol CAP
- removed C72: 1.5nF, symbol C
- removed C73: 330uF, symbol CAPAPOL
- removed C74: 100uF, symbol CAPAPOL
- removed D2: DIODESCH, symbol DIODESCH
- removed D3: DIODESCH 1 AMP, symbol DIODESCH
- removed IC1: FSUSB20, MSOP10-0.5, symbol FSUSB20
- removed J1: MICROSD12P, TFC014A-YS, symbol MICROSD12P
- removed J2: USBA_RECEPTACLE, USBA, symbol USBA_RECEPTACLE
- removed J3: USBA-PLUG, symbol USBA-PLUG
- removed L3: 170uH, symbol INDUCTOR
- removed L4: 1u, symbol INDUCTOR
- removed P2: CONN_20X2, header20x2_smd_100mil, symbol CONN_20X2
- removed P3: CONN_25X2, symbol CONN_25X2
- removed Q2: SI2305, symbol MOSFET_P
- removed R20, R21: 1.2K, symbol R
- removed R7, R8: R, symbol R
- removed RP1, RP2: 22, symbol R_PACK4
- removed U1: IMX23, fpBGA169, symbol IMX23
- removed U4: MC34063, symbol MC34063
- removed X2: 32.768 KHz, symbol CRYSTAL
- added C1, C2, C3, C5: 0.1uF, symbol C
- added C4: .1uF, symbol C
- added D2, D3, D4, D5: LED, symbol LED
- added IC1: iMX233, symbol iMX233
- added J1: MICROSD, symbol MICROSD
- added J2: JACK-PLUG0, con-jack-SPC4077, symbol JACK-PLUG0
- added JP1, JP2, JP3: JUMPER, symbol JUMPER
- added P1: CONN_8X2, symbol CONN_8X2
- added P2: CONN_12X2, symbol CONN_12X2
- added P4: CONN_4X2, symbol CONN_4X2
- added P6: CONN_2, symbol CONN_2
- added R33: 0, symbol R
- added U1: ADM3101E, symbol ADM3101E
- L2: value 15uH -> HZ0805D152R-10 (1500 ohm)
- R11, R12, R14: value 47K -> 1.5k
- R13, R16: value 1K -> 1k
- R15: value 47K -> 11k
- R17, R18, R19: value 1.2K -> 11k
- R28: value 0.22 -> 1k
- R29: value 180 -> 47k
- R30: value 10K -> 1k
- R31: value 30K -> 1k
- R32: value 100K -> 47k
- R9: value R -> 1k
Connections:
- net labels added: D03, GPMI_RDN, GPMI_RDY0, GPMI_RDY1, GPMI_WPN, GPMI_WRN, LCD_D04, LCD_D05, LCD_D06, LCD_D07, RX, TX
- net labels removed: BATT5V, DMa, DMb, DPa, DPb, GNDPWR, GPMI_CE2N, GPMI_D08, GPMI_D09, GPMI_D10, GPMI_D11, GPMI_D12, GPMI_D13, GPMI_D14, GPMI_D15, HPL, HPR, HP_VGND, LCD_D10, LCD_D11, LCD_D12, LCD_D13, LCD_D14, LCD_D15, LCD_D16, LCD_D17, LCD_D8, LCD_D9, LRADC2, LRADC3, LRADC4, LRADC5, PWM3, RTC_XTAL0, RTC_XTAL1, SPEAKERN, SPEAKERP, SSPI_DATA4, UART1_RX, UART1_TX, V_OUT
- wire segments 494 -> 363
Other:
- note added: "ADM3101E CIRCUIT"
- note added: "MICRO_SD"
- note added: "Power Supply"
- note added: "UART CONNECTOR"
- note added: "USB CONNECTOR"
- note removed: "5V BUS"
- note removed: "BUS/BATT SWITCH"
- note removed: "CRYSTAL'S CIRCUIT"
- note removed: "SPI SD"
- note removed: "TAKEWING - TFC014x-YS\nhttp://downloads.qi-hardware.com/hardware/qi_avt2/v1.0/datasheet/J1~TFC014x-YS(090122).pdf"
- note removed: "USB HOST AND DEVICE"
- note removed: "http://www.molex.com/pdm_docs/sd/480372200_sd.pdf"
- moved on the sheet: BT1, C22, C23, C24, C25, C26, C27, C28, C29, C30, C31, C32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

Commit message: conectando mas senales
Parts:
- removed P1: CONN_8X2, symbol CONN_8X2
- added P1: CONN_12X2, symbol CONN_12X2
- P2: footprint (none) -> CONN_12X2
Connections:
- net labels added: HPL, HPR, VDAC1
- wire segments 363 -> 373
- no-connect marks 18 -> 20
Other:
- moved on the sheet: D3, D4, J2, P2, P6, R28, R30

Commit message: 2 mounting points has been added
Parts:
- added P3, P5: CONN_1, MJOLE, symbol CONN_1
Connections:
- wire segments 373 -> 376

Commit message: power jack changed
Parts:
- J2: footprint con-jack-SPC4077 -> JACK
Changed lines of the file:
@@
-EESchema Schematic File Version 2  date Mon 08 Aug 2011 06:51:46 AM COT
+EESchema Schematic File Version 2  date Mon 08 Aug 2011 07:05:33 AM COT
 LIBS:con-jack
 LIBS:adm3101e
@@
 F 0 "J2" H 9550 5600 50  0000 L BNN
 F 1 "JACK-PLUG0" H 9550 5200 50  0000 L BNN
-F 2 "con-jack-SPC4077" H 9850 5550 50  0001 C CNN
+F 2 "JACK" H 9850 5550 50  0001 C CNN
 	1    9850 5400
 	1    0    0    -1

Commit message: Cambios en los footprints, adición de conectores USB host, organización de señales en los conectores
Parts:
- removed R26, R5: 10K, symbol R
- removed R27: 22, symbol R
- removed RP3, RP4, RP5: 22, symbol R_PACK4
- removed SW1: SW_PUSH, symbol SW_PUSH
- added C17: 1uF, symbol C
- added L8: HZ0805D152R-10 (1500 ohm), symbol INDUCTOR
- Q1: footprint (none) -> SOT363_PHILIPS
- U1: footprint (none) -> QSOP16
Connections:
- net labels added: MIC
- net labels removed: LCD_D00, LCD_D01, LCD_D02, LCD_D03, LCD_D04, LCD_D05, LCD_D06, LCD_D07, LCD_ENABLE1
- wire segments 376 -> 371
- no-connect marks 20 -> 8
Other:
- note removed: "USB FIRMWARE RECOVERY"

Commit message: Adición de conectores USB host, conexión de HP_GND a un conector externo, Cambio de los footprints dela DDR memoria SPI, Q1,
Parts:
- removed J2: JACK-PLUG0, JACK, symbol JACK-PLUG0
- removed P3, P5: CONN_1, MJOLE, symbol CONN_1
- added J2: POWER_5V, symbol CONN_3
Connections:
- net labels added: HP_VGND
- wire segments 371 -> 368
- no-connect marks 8 -> 9
