File: PCB/i.mx233stamp/i.MX233.sch (KiCad schematic (older format))
At the start: 86 parts, among them IC1 iMX233, J1 MICROSD, J2 POWER_5V, P1 CONN_12X2, P2 CONN_12X2, P4 CONN_4X2, P6 CONN_2, Q1 MMDT3904, SW2 SW_PUSH, SW3 SW_PUSH, U1 ADM3101E, X1 24 MHz

Commit message: nuevo cristal
Parts:
- removed X1: 24 MHz, symbol CRYSTAL
- added X1: 24MHz, ABM8G, symbol ABM8G
Connections:
- wire segments 368 -> 371

Commit message: Adición del footprint del m25pxx, y re-organización del layout de la placa
Parts:
- removed R33: 0, symbol R
Connections:
- wire segments 371 -> 370

Commit message: cambios menoresn la ddr
Parts:
- added P3, P5: CONN_1, MHOLE, symbol CONN_1
Connections:
- net labels added: GND_CASE
- wire segments 370 -> 373
