File: PCB/i.mx233stamp/i.mx233stamp.sch (KiCad schematic (older format))
At the start: 0 parts

Commit message: clean-up
Connections:
- wire segments 20 -> 22
Changed lines of the file:
@@
-EESchema Schematic File Version 2  date mié 02 feb 2011 14:04:32 COT
+EESchema Schematic File Version 2  date Fri 05 Aug 2011 02:31:32 PM COT
+LIBS:con-jack
+LIBS:adm3101e
+LIBS:microsd
 LIBS:transistor-npn
 LIBS:ipc-7351-transistor
@@
 LIBS:PWR
 LIBS:m25p32
+LIBS:PROpendous-cache
 LIBS:w_analog
+LIBS:gl850g
+LIBS:srf2012
 LIBS:i.mx233stamp-cache
-EELAYER 24  0
+EELAYER 25  0
 EELAYER END
 $Descr A4 11700 8267
-Sheet 1 3
+encoding utf-8
+Sheet 1 4
 Title ""
-Date "2 feb 2011"
+Date "5 aug 2011"
 Rev ""
 Comp ""
@@
 $EndDescr
 Wire Wire Line
-	4750 2150 5250 2150
+	3000 3550 3150 3550
 Wire Wire Line
-	4750 1850 5250 1850
+	4750 1650 5250 1650
+Wire Wire Line
+	4750 2250 5250 2250
+Wire Wire Line
+	5250 1950 4750 1950
+Wire Wire Line
+	5250 1750 4750 1750
+Wire Bus Line
+	5250 2400 4750 2400
+Wire Wire Line
+	4750 3450 5250 3450
+Wire Wire Line
+	5250 3200 4750 3200
+Wire Wire Line
+	4750 2950 5250 2950
+Wire Wire Line
+	4750 4050 5250 4050
+Wire Wire Line
+	4750 3800 5250 3800
+Wire Wire Line
+	4750 3600 5250 3600
+Wire Wire Line
+	4750 2850 5250 2850
+Wire Wire Line
+	4750 2750 5250 2750
+Wire Wire Line
+	4750 2650 5250 2650
+Wire Wire Line
+	4750 3700 5250 3700
+Wire Wire Line
+	4750 3950 5250 3950
+Wire Wire Line
+	4750 3100 5250 3100
+Wire Wire Line
+	5250 3350 4750 3350
+Wire Wire Line
+	4750 2050 5250 2050
 Wire Bus Line
 	4750 2500 5250 2500
 Wire Wire Line
-	4750 2050 5250 2050
+	4750 1850 5250 1850
 Wire Wire Line
-	5250 3350 4750 3350
+	4750 2150 5250 2150
 Wire Wire Line
-	4750 3100 5250 3100
-Wire Wire Line
-	4750 3950 5250 3950
-Wire Wire Line
-	4750 3700 5250 3700
-Wire Wire Line
-	4750 2650 5250 2650
-Wire Wire Line
-	4750 2750 5250 2750
-Wire Wire Line
-	4750 2850 5250 2850
-Wire Wire Line
-	4750 3600 5250 3600
-Wire Wire Line
-	4750 3800 5250 3800
-Wire Wire Line
-	4750 4050 5250 4050
-Wire Wire Line
-	4750 2950 5250 2950
-Wire Wire Line
-	5250 3200 4750 3200
-Wire Wire Line
-	4750 3450 5250 3450
-Wire Bus Line
-	5250 2400 4750 2400
-Wire Wire Line
-	5250 1750 4750 1750
-Wire Wire Line
-	5250 1950 4750 1950
-Wire Wire Line
-	5250 2300 5250 2250
-Wire Wire Line
-	5250 2250 4750 2250
+	3150 3450 3000 3450
+$Sheet
+S 2150 3250 850  850
+U 4E3BEC51
+F0 "USB" 60
+F1 "USB.sch" 60
+F2 "USB_DM0" T R 3000 3550 60
+F3 "USB_DP0" T R 3000 3450 60
+$EndSheet
 $Sheet
 S 5250 1600 1150 2500
@@
 F15 "DDR_RASN" I L 5250 2950 60
 F16 "DDR_WEN" I L 5250 2750 60
-F17 "SSPI_DATA4" I L 5250 2050 60
-F18 "SSPI_DATA2" I L 5250 1950 60
-F19 "SSPI_SCK" I L 5250 2150 60
-F20 "SSPI_CMD" I L 5250 2250 60
-F21 "SSPI_DATA1" I L 5250 1850 60
-F22 "SSPI_DATA0" I L 5250 1750 60
+F17 "GPMI_D04" I L 5250 2050 60
+F18 "GPMI_D02" I L 5250 1950 60
+F19 "GPMI_WRN" I L 5250 2150 60
+F20 "GPMI_RDY1" I L 5250 2250 60
+F21 "GPMI_D01" I L 5250 1850 60
+F22 "GPMI_D00" I L 5250 1750 60
+F23 "GPMI_D03" I L 5250 1650 60
 $EndSheet
 $Sheet
@@
 F15 "DDR_BA1" O R 4750 4050 60
 F16 "DDR_BA0" O R 4750 3950 60
-F17 "SSPI_DATA4" O R 4750 2050 60
-F18 "SSPI_SCK" O R 4750 2150 60
-F19 "SSPI_CMD" O R 4750 2250 60
-F20 "SSPI_DATA0" O R 4750 1750 60
-F21 "SSPI_DATA1" O R 4750 1850 60
-F22 "SSPI_DATA2" O R 4750 1950 60
+F17 "GPMI_D04" O R 4750 2050 60
+F18 "GPMI_WRN" O R 4750 2150 60
+F19 "GPMI_RDY1" O R 4750 2250 60
+F20 "GPMI_D00" O R 4750 1750 60
+F21 "GPMI_D01" O R 4750 1850 60
+F22 "GPMI_D02" O R 4750 1950 60
+F23 "GPMI_D03" O R 4750 1650 60
+F24 "USB_DM" B L 3150 3550 60
+F25 "USB_DP" B L 3150 3450 60
 $EndSheet
 $EndSCHEMATC
